File: PCB/LPP MainBoard Gen_1_Ver_1.brd (EAGLE design)
At the start: 50 x 115 mm, 48 parts, among them IC1 FE1.1S, U1 MAX15070, U3 BTN7933B, U4 MAX15070, U5 BTN7933B, U7 Pill STM32G431, U8 Blue Pill STM32F103

Commit message: modified:   LPP_STM32F103Cx/MDK-ARM/JLinkLog.txt 	modified:   LPP_STM32F103Cx/MDK-ARM/LPP_STM32F103Cx.uvguix.user 	modified:   PCB/LPP MainBoard Gen_1_Ver_1.brd 	modified:   PCB/LPP_MainBoard_Gen_1_Ver_1.dip
Parts:
- moved CNC 7.70 mm to (44.3, 52.0)
- moved STEPPER_SHIELD 6.90 mm to (39.1, 51.2)
- moved BLDC 6.70 mm to (38.1, 105.4)
- moved DC 6.70 mm to (46.0, 105.4)
- moved R5 6.70 mm to (36.8, 85.7)
- moved R6 6.70 mm to (36.8, 92.7)
- moved R8 6.70 mm to (36.8, 89.2)
- moved U3 6.70 mm to (39.9, 83.5)
- moved U5 6.70 mm to (39.9, 93.8)
- moved R3 6.70 mm to (36.8, 82.1)
- moved R9 6.70 mm to (36.8, 96.1)
- moved C1 5.30 mm to (29.0, 106.0)
- moved FPC 4.90 mm to (24.3, 115.7)
- moved LAZER_CP 4.24 mm to (8.70, 109.1)
- moved R4 3.40 mm to (5.40, 103.9)
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Routing:
- net Сеть_7: track 279.0 -> 305.6 mm
- net Сеть_16: track 151.2 -> 176.9 mm
- net Сеть_0: track 574.3 -> 592.2 mm, vias 20 -> 21
- net Сеть_33: track 141.6 -> 150.9 mm
- net Сеть_6: track 132.1 -> 140.4 mm
- net Сеть_29: track 72.6 -> 79.5 mm
- net Сеть_20: track 40.4 -> 34.1 mm
- net Сеть_34: track 98.0 -> 104.1 mm
- net Сеть_36: track 32.9 -> 26.8 mm
- net Сеть_19: track 42.8 -> 48.8 mm
- net Сеть_35: track 90.7 -> 96.7 mm
- net Сеть_13: track 44.9 -> 39.4 mm
- net Сеть_12: track 76.9 -> 81.8 mm
- net Сеть_14: track 78.8 -> 83.7 mm
- net Сеть_22: track 61.7 -> 57.1 mm
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Other:
- board size 50 x 115 mm -> 50 x 120 mm
